Commit message: update config

File: beckhoff_testbed_description/urdf/el1859_ros2_control.xacro (robot description, xacro)
@@ -1,5 +1,5 @@
 <?xml version="1.0"?>
 <robot xmlns:xacro="http://www.ros.org/wiki/xacro">
-  <xacro:macro name="GPIO_ros2_control" params="name:=''">
+  <xacro:macro name="el1859" params="name:=''">
       <gpio name="gpio">
         <command_interface name="do0"/>

File: beckhoff_testbed_description/urdf/ethercat_ros2_control.xacro (robot description, xacro)
@@ -17,8 +17,8 @@
         </xacro:unless>
       </hardware>
-       <xacro:include filename="$(find beckhoff_testbed_description)/urdf/GPIO_ros2_control.xacro"/>
-       <xacro:GPIO_ros2_control name="${name}_gpio"/>
+       <xacro:include filename="$(find beckhoff_testbed_description)/urdf/el1859_ros2_control.xacro"/>
+       <xacro:el1859 name="${name}_el1859"/>
        <xacro:include filename="$(find beckhoff_testbed_description)/urdf/el7201_ros2_control.xacro"/>
-       <xacro:el7201 name="${name}_gpio"/>
+       <xacro:el7201 name="${name}_el7201"/>
     </ros2_control>
   </xacro:macro>

File: beckhoff_testbed_description/urdf/main.xacro (robot description, xacro)
@@ -1,4 +1,4 @@
 <?xml version="1.0"?>
-<robot name="battery_cell" xmlns:xacro="http://www.ros.org/wiki/xacro">
+<robot name="beckhoff_testbed" xmlns:xacro="http://www.ros.org/wiki/xacro">
   <xacro:arg name="use_ethercat_fake_hardware" default="false"/>
   <!-- Include ROS2 HW interface definitions for GPIO modules -->
